File: fuente.kicad_sch (KiCad schematic)
At the start: 15 parts, among them J3 Screw_Terminal_01x02, Q4 IRLZ44N, U7 LM2596S-5

Commit message: Agregar protección de sobre tensión/tensión inversa (3)
Connections:
- net LProt renamed LPROT
Changed lines of the file:
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@@
 		)
 	)
-	(label "LProt"
+	(label "LPROT"
 		(at 130.81 88.9 0)
 		(effects
