File: fuente.kicad_sch (KiCad schematic)
At the start: 15 parts, among them J3 Screw_Terminal_01x02, Q4 IRLZ44N, U7 LM2596S-5

Commit message: Cambiar agujeros de placa, invertir terminales de fuente
Connections:
- net GND: now also J3.1 (Pin_1); no longer J3.2 (Pin_2)
- net at TH1.1: now also J3.2 (Pin_2); no longer J3.1 (Pin_1)
Other:
- moved on the sheet: J3
Changed lines of the file:
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@@
 	(symbol
 		(lib_id "Connector:Screw_Terminal_01x02")
-		(at 67.31 88.9 0)
-		(mirror y)
+		(at 67.31 91.44 180)
 		(unit 1)
 		(exclude_from_sim no)
@@
 		(dnp no)
 		(property "Reference" "J3"
-			(at 67.31 83.82 0)
+			(at 67.31 96.52 0)
 			(effects
 				(font
@@
 		)
 		(property "Footprint" "TerminalBlock_Phoenix:TerminalBlock_Phoenix_MKDS-1,5-2_1x02_P5.00mm_Horizontal"
-			(at 67.31 88.9 0)
+			(at 67.31 91.44 0)
 			(effects
 				(font
@@
 		)
 		(property "Datasheet" "~"
-			(at 67.31 88.9 0)
+			(at 67.31 91.44 0)
 			(effects
 				(font
@@
 		)
 		(property "Description" "Generic screw terminal, single row, 01x02, script generated (kicad-library-utils/schlib/autogen/connector/)"
-			(at 67.31 88.9 0)
+			(at 67.31 91.44 0)
 			(effects
 				(font

Commit message: Actualizar zener a 1N4752A (33V)
Parts:
- D12: value 1N47xxA -> 1N4752A
Changed lines of the file:
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@@
 			)
 		)
-		(property "Value" "1N47xxA"
+		(property "Value" "1N4752A"
 			(at 107.95 96.5199 90)
 			(effects
